File: hardware/MidiFaderLite/MidiFaderLite.kicad_pcb (KiCad board)
At the start: 2 copper layers, 260 x 159 mm, 19 parts, among them SW1 Rotary_Encoder_Switch, SW2 Rotary_Encoder_Switch, SW3 Rotary_Encoder_Switch, SW4 Rotary_Encoder_Switch, SW5 SW_SPST, SW6 SW_SPST, SW7 SW_SPST, SW8 SW_SPST, U1 Teensy++2.0_(Arduino), U2 L293D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

Commit message: Update schematic with latest plan
Parts:
- removed MF4: MFader, Moving_fader:MFader
- removed RV4: R_POT, Potentiometer_THT:Potentiometer_Alps_RK097_Single_Horizontal
- removed SW6, SW7, SW8: SW_SPST, Button_Switch_THT:SW_DIP_SPSTx01_Slide_9.78x4.72mm_W7.62mm_P2.54mm
- added D1: LED_CRGB, LED_THT:LED_D5.0mm-4_RGB, F.Cu at (225.0, -15.3)
- added R1: R_Small, Resistor_THT:R_Axial_DIN0207_L6.3mm_D2.5mm_P10.16mm_Horizontal, F.Cu at (163.9, -89.0)
- added R10: R_Small, Resistor_THT:R_Axial_DIN0207_L6.3mm_D2.5mm_P10.16mm_Horizontal, F.Cu at (177.2, -85.0)
- added R11: R_Small, Resistor_THT:R_Axial_DIN0207_L6.3mm_D2.5mm_P10.16mm_Horizontal, F.Cu at (163.9, -76.8)
- added R12: R_Small, Resistor_THT:R_Axial_DIN0207_L6.3mm_D2.5mm_P10.16mm_Horizontal, F.Cu at (177.2, -80.9)
- added R13: R_Small, Resistor_THT:R_Axial_DIN0207_L6.3mm_D2.5mm_P10.16mm_Horizontal, F.Cu at (177.2, -76.8)
- added R2: R_Small, Resistor_THT:R_Axial_DIN0207_L6.3mm_D2.5mm_P10.16mm_Horizontal, F.Cu at (217.9, -61.0)
- added R3: R_Small, Resistor_THT:R_Axial_DIN0207_L6.3mm_D2.5mm_P10.16mm_Horizontal, F.Cu at (163.9, -85.0)
- added R4: R_Small, Resistor_THT:R_Axial_DIN0207_L6.3mm_D2.5mm_P10.16mm_Horizontal, F.Cu at (164.3, -68.0)
- added R5: R_Small, Resistor_THT:R_Axial_DIN0207_L6.3mm_D2.5mm_P10.16mm_Horizontal, F.Cu at (164.3, -64.0)
- added R6: R_Small, Resistor_THT:R_Axial_DIN0207_L6.3mm_D2.5mm_P10.16mm_Horizontal, F.Cu at (177.6, -68.0)
- added R7: R_Small, Resistor_THT:R_Axial_DIN0207_L6.3mm_D2.5mm_P10.16mm_Horizontal, F.Cu at (164.3, -59.9)
- added R8: R_Small, Resistor_THT:R_Axial_DIN0207_L6.3mm_D2.5mm_P10.16mm_Horizontal, F.Cu at (177.2, -89.0)
- added R9: R_Small, Resistor_THT:R_Axial_DIN0207_L6.3mm_D2.5mm_P10.16mm_Horizontal, F.Cu at (163.9, -80.9)
- added U4: Teensy3.2, KiCad_library:Teensy30_31_32_LC, F.Cu at (182.2, -18.0)
- RV1, RV2, RV3: footprint Potentiometer_THT:Potentiometer_Alps_RK097_Single_Horizontal -> Potentiometer_THT:Potentiometer_Alps_RK09L_Single_Vertical
- SW1: value Rotary_Encoder_Switch -> Rotary_Encoder; footprint Rotary_Encoder:RotaryEncoder_Alps_EC11E-Switch_Vertical_H20mm -> Rotary_Encoder:RotaryEncoder_Alps_EC11E_Vertical_H20mm
- SW2, SW3, SW4: value Rotary_Encoder_Switch -> SW_SPST; footprint Rotary_Encoder:RotaryEncoder_Alps_EC11E-Switch_Vertical_H20mm -> Button_Switch_THT:SW_DIP_SPSTx01_Slide_9.78x4.72mm_W7.62mm_P2.54mm
- moved U2 166.0 mm to (265.0, -29.6)
- moved U3 166.0 mm to (249.2, -30.4)
- moved RV2 156.1 mm to (251.6, -94.8)
- moved SW5 153.8 mm to (189.4, -62.8)
- moved RV3 153.2 mm to (225.5, -80.3)
- moved U1 151.3 mm to (321.0, 55.6), turned to 270 degrees
- moved RV1 146.9 mm to (251.8, -76.5)
- moved SW4 112.4 mm to (176.1, -54.6)
- moved SW2 106.4 mm to (178.0, -62.8)
- moved MF1 100.6 mm to (128.0, 67.5), turned to 180 degrees
- moved SW3 87.3 mm to (164.7, -54.6)
- moved MF2 77.5 mm to (128.0, 92.5), turned to 180 degrees
- moved SW1 71.4 mm to (227.3, -42.5)
- moved MF3 62.4 mm to (128.0, 117.5), turned to 180 degrees
Connections:
- net RA1 renamed ROTA
- net RB1 renamed ROTB
- MF1 pad 3: VDD -> +5V
- MF1 pad 6: (no net) -> Net-(MF1-Pad6)
- MF2 pad 3: VDD -> +5V
- MF2 pad 6: (no net) -> Net-(MF2-Pad6)
- MF3 pad 3: VDD -> +5V
- MF3 pad 6: (no net) -> Net-(MF3-Pad6)
- RV1 pad 3: VDD -> +5V
- RV2 pad 3: VDD -> +5V
- RV3 pad 3: VDD -> +5V
- SW5 pad 1: ControlSwitch1 -> GNDREF
- SW5 pad 2: GNDREF -> Button4
- U1 pad 21: (no net) -> +5V
- U1 pad 24: POT4 -> POT1
- U1 pad 25: POT3 -> POT2
- U1 pad 26: POT2 -> POT3
- U1 pad 27: POT1 -> (no net)
- U1 pad 28: Slider4 -> (no net)
- U1 pad 34: RA2 -> (no net)
- U1 pad 35: RB2 -> (no net)
- U1 pad 36: (no net) -> Button1
- U1 pad 37: (no net) -> Button2
- U1 pad 38: DIRBFadeur4 -> Button3
- U1 pad 39: DIRAFadeur4 -> Button4
- U1 pad 40: SpeedFadeur4 -> LED_BLUE
- U1 pad 41: (no net) -> LED_GREEN
- U1 pad 42: (no net) -> LED_RED
- U1 pad 43: VDD -> +5V
- U1 pad 44: ControlSwitch4 -> Touch1
- U1 pad 45: ControlSwitch3 -> Touch2
- U1 pad 46: ControlSwitch2 -> Touch3
- U1 pad 47: ControlSwitch1 -> (no net)
- U1 pad 48: RS1 -> (no net)
- U1 pad 49: RS2 -> (no net)
- U1 pad 5: RA4 -> (no net)
- U1 pad 50: RS3 -> (no net)
- U1 pad 51: RS4 -> (no net)
- U1 pad 6: RB4 -> (no net)
- U2 pad 16: VDD -> +5V
- U3 pad 10: DIRAFadeur4 -> (no net)
- U3 pad 11: Net-(MF4-Pad4) -> (no net)
- U3 pad 14: Net-(MF4-Pad5) -> (no net)
- U3 pad 15: DIRBFadeur4 -> (no net)
- U3 pad 16: VDD -> +5V
- U3 pad 9: SpeedFadeur4 -> (no net)
Other:
- board size 260 x 159 mm -> 190 x 100 mm
